File: SatUplink/SatUplink-v12.sch (EAGLE design)
At the start: 40 parts, among them U1 MIC5219-3.3, U2 AP7311-1.8, U3 74HC5040, U4 SPOT-CONNECT, U5 ARDUINO_SHIELD, U6 MIC5219-3.0, U7 MIC5219-3.0

Commit message: Fixing schematic typo.
Parts:
- U3: value 74HC5040 -> 74HC4050
Changed lines of the file:
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@@
 <part name="C12" library="SparkFun" deviceset="CAP_POL" device="1206" value="10uF"/>
 <part name="GND16" library="SparkFun" deviceset="GND" device=""/>
-<part name="U3" library="SparkFun" deviceset="HEX_CONVERTER" device="" value="74HC5040"/>
+<part name="U3" library="SparkFun" deviceset="HEX_CONVERTER" device="" value="74HC4050"/>
 <part name="GND17" library="SparkFun" deviceset="GND" device=""/>
 <part name="P+7" library="SparkFun" deviceset="3.3V" device=""/>
