File: SatUplink/SatUplink-v12.brd (EAGLE design)
At the start: 55 x 68 mm, 40 parts, among them U1 MIC5219-3.3, U2 AP7311-1.8, U3 74HC5040, U4 SPOT-CONNECT, U5 ARDUINO_SHIELD, U6 MIC5219-3.0, U7 MIC5219-3.0

Commit message: Fixing schematic typo.
Parts:
- U3: value 74HC5040 -> 74HC4050
